File: neuron.kicad_sch (KiCad schematic)
At the start: 67 parts, among them J1 Conn_01x03, J2 Conn_01x03, J3 Conn_01x03, J4 Conn_02x03, Q1 BSS84, Q2 2N7002, Q3 BSS84, Q4 2N7002, Q5 BSS84, Q6 2N7002, Q7 2N7002, Q8 2sk3018, U1 74HC14, U4 MCP6001-OT, U5 LM339, U6 LM339

Commit message: Update for second production run
Parts:
- D2, D3, D4, D5, D6, D7: LCSC C779450 -> C917185
- R12, R13, R14, R15, R16, R17, R26: value 100k -> 56k; LCSC C25741 -> C25796
- R20, R21, R22, R23, R24, R25: value 100 -> 150; LCSC C25076 -> C25082
- R30: value 33 -> 10; LCSC C25105 -> C25077
- RV1: value 20k -> 5k
- RV4: value 200k -> 100k; LCSC C128551 -> C128545

Commit message: Migrate to KiCad 7
Parts:
- BT1: value Battery_Cell -> ${SIM.PARAMS}; Spice_Netlist_Enabled N -> (none); Spice_Primitive R -> (none)
- D1, D2, D3, D4, D5, D6, D7: Spice_Lib_File ./models/led.mod -> (none); Spice_Model YELLOW -> (none); Spice_Netlist_Enabled Y -> (none); Spice_Node_Sequence 2 1 -> (none); Spice_Primitive D -> (none)
- J1, J2, J3: Spice_Lib_File ./models/pin-header.mod -> (none); Spice_Model pins -> (none); Spice_Netlist_Enabled Y -> (none); Spice_Primitive X -> (none)
- J4: Spice_Lib_File ./models/pin-header.mod -> (none); Spice_Model pins -> (none); Spice_Netlist_Enabled N -> (none); Spice_Primitive X -> (none)
- Q1, Q3, Q5: Spice_Lib_File ./models/bss84.mod -> (none); Spice_Model BSS84 -> (none); Spice_Netlist_Enabled Y -> (none); Spice_Primitive X -> (none)
- Q2, Q4, Q6, Q7, Q8: Spice_Lib_File ./models/2sk3018.mod -> (none); Spice_Model 2SK3018 -> (none); Spice_Netlist_Enabled Y -> (none); Spice_Primitive X -> (none)
- RV1, RV2, RV3: Spice_Lib_File ./models/poti.mod -> (none); Spice_Model pot value=20k ratio=0.5 -> (none); Spice_Netlist_Enabled Y -> (none); Spice_Primitive X -> (none)
- RV4: Spice_Lib_File ./models/poti.mod -> (none); Spice_Model pot value=200k ratio=0.3 -> (none); Spice_Netlist_Enabled Y -> (none); Spice_Primitive X -> (none)
- RV5: Spice_Lib_File ./models/poti.mod -> (none); Spice_Model pot value=200k ratio=0.95 -> (none); Spice_Netlist_Enabled Y -> (none); Spice_Primitive X -> (none)
- U1: Spice_Lib_File ./models/sn74hc14.mod -> (none); Spice_Model SN74HC14 -> (none); Spice_Netlist_Enabled Y -> (none); Spice_Primitive X -> (none)
- U4: Spice_Lib_File ./models/mcp6001.mod -> (none); Spice_Model MCP6001 -> (none); Spice_Netlist_Enabled Y -> (none); Spice_Primitive X -> (none)
- U5, U6: Spice_Lib_File ./models/lm339.mod -> (none); Spice_Model LM339 -> (none); Spice_Netlist_Enabled Y -> (none); Spice_Primitive X -> (none)
- V1: Spice_Model pulse(2.7 0 2n 2n 2n 20m 100m) -> (none); Spice_Netlist_Enabled Y -> (none); Spice_Primitive V -> (none)
- V2: value 2.7 -> 2.0; Spice_Model dc(2.0) -> (none); Spice_Netlist_Enabled Y -> (none); Spice_Primitive V -> (none)

Commit message: Implement exponential synapses
Co-authored-by: Yannik Stradmann <yannik@stradmann.name>
Co-authored-by: Julian Göltz <mail@julian-goeltz.de>
Parts:
- removed J1, J2, J3: Conn_01x03, Connector_PinHeader_2.54mm:PinHeader_1x03_P2.54mm_Vertical, symbol Connector_Generic:Conn_01x03
- removed Q1, Q3: BSS84, Package_TO_SOT_SMD:SOT-23, symbol Transistor_FET:BSS84
- removed Q4, Q6, Q7: 2N7002, Package_TO_SOT_SMD:SOT-23, symbol Transistor_FET:2N7002
- removed R19: 100k, Resistor_SMD:R_0402_1005Metric, symbol Device:R_Small
- removed U1: 74HC14, Package_SO:TSSOP-14_4.4x5mm_P0.65mm, symbol 74xx:74HC14
- removed U4: MCP6001-OT, Package_TO_SOT_SMD:SOT-23-5, symbol Amplifier_Operational:MCP6001-OT
- added C1, C8: 100n, Capacitor_SMD:C_0402_1005Metric, symbol Device:C_Small
- added C2: 10u ic=0.0, Capacitor_SMD:C_0402_1005Metric, symbol Device:C_Small
- added J1, J2, J3: Conn_02x01, Connector_PinHeader_2.54mm:PinHeader_1x02_P2.54mm_Vertical, symbol Connector_Generic:Conn_02x01
- added Q1, Q10, Q11, Q12, Q3: 2sk3018, Package_TO_SOT_SMD:SOT-23, symbol Transistor_FET:2N7002
- added Q4, Q6: BSS84, Package_TO_SOT_SMD:SOT-23, symbol Transistor_FET:BSS84
- added Q7: SI2301, Package_TO_SOT_SMD:SOT-23, symbol Transistor_FET:BSS84
- added Q9: 2N7002, Package_TO_SOT_SMD:SOT-23, symbol Transistor_FET:2N7002
- added R10, R13, R22, R23, R25, R7, R8: 22k, Resistor_SMD:R_0402_1005Metric, symbol Device:R_Small
- added R12: 47k, Resistor_SMD:R_0402_1005Metric, symbol Device:R_Small
- added R14, R15: 2.2k, Resistor_SMD:R_0402_1005Metric, symbol Device:R_Small
- added R16, R42, R9: 470, Resistor_SMD:R_0402_1005Metric, symbol Device:R_Small
- added RV4: 20k, Custom:Potentiometer, symbol Device:R_Potentiometer_Small
- added SW1, SW2, SW3: SW_SPDT, Custom:K3-1290S-E1, symbol Switch:SW_SPDT
- added U1: MCP6004, Package_SO:TSSOP-14_4.4x5mm_P0.65mm, symbol Amplifier_Operational:MCP6004
- BT1: value ${SIM.PARAMS} -> type="R" model="Battery_Cell" lib=""
- C5: renamed from C1; value 4.7u -> 22u ic=0.6; footprint Capacitor_SMD:C_0805_2012Metric -> Capacitor_SMD:C_0402_1005Metric; LCSC C1779 -> C2836678
- C9: renamed from C2; value 1u -> 1u ic=2; footprint Capacitor_SMD:C_0805_2012Metric -> Capacitor_SMD:C_0402_1005Metric; LCSC C28323 -> C52923
- D1: LCSC C779450 -> C779448
- D2, D3, D4, D5, D6, D7: LCSC C917185 -> C779448
- Q2: value 2N7002 -> 2sk3018; LCSC C8545 -> C181084
- Q8: value 2sk3018 -> SI2302; LCSC C181084 -> C10488
- R11: value 100k -> 47k; LCSC C25741 -> C5152005
- R4, R5, R6: value 100k -> 10k; LCSC C25741 -> C25744
- RV1: LCSC C128550 -> C128557
- RV2, RV3: value 20k -> 5k; LCSC C128550 -> C128557
- RV6: renamed from RV5; value 200k -> 50k; LCSC C128551 -> C145161
- V2: value 2.0 -> 2
- renumbered C5 to C6, C6 to C7, R8 to R17, R26 to R18, R7 to R19, R18 to R20, R9 to R21, R27 to R24, R28 to R26, R29 to R27, R10 to R28, R12 to R29, R13 to R30, R14 to R31, R15 to R32, R16 to R33, R17 to R34, R20 to R35, R21 to R36, R22 to R37, R23 to R38, R24 to R39, R25 to R40, R30 to R41, RV4 to RV5, U5 to U2, U6 to U3
Connections:
- net EXC3 is gone; now on net VDD: R5.1
- net INH1 is gone; now on an unnamed net: Q2.1 (G), R2.1
- net INH2 is gone; now on net VDD: R4.1
- net INH3 is gone; now on net VDD: R6.1
- net GND: now also C9.2, C1.1, C8.1, J1.1 (Pin_1), J2.1 (Pin_1), J3.1 (Pin_1), Q1.2 (S), Q10.2 (S), Q11.2 (S), Q12.2 (S), Q3.2 (S), Q9.2 (S), R13.2, R15.2, R23.2, R8.2, U1.11 (V-); no longer C9.1, Q8.2 (S), R4.2, R5.2, R6.2
- net MEM: now also Q8.3 (D), Q7.3 (D); no longer RV1.2, RV1.3, RV2.2, RV2.3, RV3.2, RV3.3
- net REFR: now also C9.1; no longer C9.2
- net RESET: now also Q12.1 (G), Q9.1 (G)
- net SPK: now also Q10.3 (D), Q11.1 (G), R25.1; no longer Q8.1 (G)
- net VDD: now also Q4.2 (S), Q6.2 (S), R10.1, R14.1, R22.1, R25.2, R7.1, U1.4 (V+); no longer R11.1
- net VU7: now also Q12.3 (D)
- net at V1.1: now also J2.2 (Pin_2)
- net at RV2.1: now also Q5.3 (D), SW2.3 (C)
- net at U3.5 (+): now also C8.2, R22.2, R23.1; no longer R11.2
- net at R21.2, R24.1, U3.1: now also Q10.1 (G)
- net at R19.2: now also Q9.3 (D)
- net at Q2.3 (D): now also SW2.2 (B); no longer RV1.1
- net at R26.1: now also Q11.3 (D); no longer Q8.3 (D)
- net at Q5.1 (G): now also R5.2, SW2.1 (A)
- net at RV5.2: now also U1.3 (+)
- net at RV3.1: now also Q6.3 (D), SW3.3 (C); no longer Q5.3 (D)
- net VLEAK: now reaches RV6.3
- net VLEAK: now also U1.1, U1.2 (-)
- net EXC1: no longer names the net of R1.1
- net EXC1: now also J1.2 (Pin_2), Q1.1 (G)
- net EXC2: no longer names the net of R3.1
- net EXC2: now also J3.2 (Pin_2), Q3.1 (G)
- new net: Q4.1 (G), R4.2, SW1.3 (C)
- new net: R12.2, R13.1, U1.12 (+)
- new net: R10.2, R11.1, U1.10 (+)
- new net: Q1.3 (D), SW1.2 (B)
- new net: Q6.1 (G), R6.2, SW3.1 (A)
- new net: Q4.3 (D), RV1.1, SW1.1 (A)
- new net: C1.2, R7.2, R8.1, U1.5 (+)
- new net: R9.1, RV1.2, RV1.3
- new net: C2.1, R16.2, R42.2, R9.2, RV4.3, U1.6 (-)
- new net: R42.1, RV3.2, RV3.3
- new net: Q8.2 (S), R15.1, U1.13 (-)
- new net: Q8.1 (G), U1.14
- new net: Q3.3 (D), SW3.2 (B)
- new net: Q7.1 (G), U1.8
- new net: Q7.2 (S), R14.2, U1.9 (-)
- new net: R16.1, RV2.2, RV2.3
- new net VSYN: C2.2, R11.2, R12.1, RV4.1, RV4.2, U1.7
Other:
- note added: "ACTIVE LOW? HIGH?"
- note removed: "SYNAPSES"
- moved on the sheet: BT1, C3, C4, C5, C6, C7, C9, D1, D2, D3, D4, D5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

Commit message: Update comments in schematic
Other:
- note added: "threshold voltage (incl. hysteresis): 1/2 VDD with feedback during refr.: 1/4 VDD"
- note removed: "ACTIVE LOW? HIGH?"
- note removed: "threshold voltage (incl. hysteresis): 2/3 VDD (feedback during refr.: 1/3 VDD)"
Changed lines of the file:
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@@
     (effects (font (size 2.54 2.54) (thickness 0.508) bold) (justify left bottom))
-  )
-  (text "ACTIVE LOW? HIGH?" (at -647.7 -85.725 0)
-    (effects (font (size 100 100)) (justify left bottom))
   )
   (text "TESTBENCH (for simulation only)" (at 212.09 220.98 0)
     (effects (font (size 2.54 2.54) (thickness 0.508) bold) (justify left bottom))
   )
-  (text "threshold voltage (incl. hysteresis):\n2/3 VDD (feedback during refr.: 1/3 VDD)"
+  (text "threshold voltage (incl. hysteresis): 1/2 VDD\n         with feedback during refr.: 1/4 VDD"
     (at 281.94 59.69 0)
     (effects (font (size 1 1)) (justify left bottom))

Commit message: Clean up simulation models and testbench
Parts:
- added R43: 10, Resistor_SMD:R_0402_1005Metric, symbol Device:R_Small
- added R44: 4.7k, Resistor_SMD:R_0402_1005Metric, symbol Device:R_Small
- C2: value 10u ic=0.0 -> 10u
- C5: value 22u ic=0.6 -> 22u ic=0.5
- V2: value 2 -> 2.5
Connections:
- net VDD: now also R43.1; no longer V2.1
- net INPUT_0: now reaches J1.2 (Pin_2), Q1.1 (G), R1.1
- net INPUT_1: now reaches J2.2 (Pin_2), Q2.1 (G), R2.1
- net INPUT_1: now also R44.1; no longer V1.1
- net INPUT_3: now reaches J3.2 (Pin_2), Q3.1 (G), R3.1
- new net: R43.2, V2.1
- new net: R44.2, V1.1
Other:
- note added: ".tran 1m 5 uic"
- moved on the sheet: BT1, J4, R20, U2E, U3E, V1, V2

Commit message: Clean up schematic
Other:
- note added: "SUPPLY"
- note added: "SYNAPSES"
- note added: "SYNAPTIC INTEGRATOR"
- moved on the sheet: BT1, C1, C2, C3, C4, C5, C6, C7, C8, C9, D1, D2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
